Commit message: bringup

File: src/rubot_mecanum_description/urdf/rubot_custom.urdf (robot description, URDF)
Before this commit: robot rubot, 9 links, 8 joints
Links:
- link camera: geometry collision box size=0.05 0.05 0.025; visual mesh filename=package://rubot_mecanum_description/meshes/rubot/piCamera.s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 scale=0.001 0.001 0.001
- link part: geometry collision box size=0.05 0.05 0.025; visual box size=0.05 0.05 0.025
Joints:
- joint scan_joint: origin xyz=0 0 0.15 rpy=0 0 3.14 -> xyz=0 0 0.15 rpy=0 0 0
